Commit message: Fix link's geometry in URDF

File: urdf/hdpr.urdf (robot description, URDF)
Before this commit: robot HDPR, 26 links, 25 joints
Links:
- removed link body
- added link body_base; visual box size=1.0 0.7 0.1
- link fl_wheel: geometry visual mesh filename=package://ga_slam_visualization/urdf/meshes/exoter/wheel.stl scale=1.66 1 1.66
- link fr_wheel: geometry visual mesh filename=package://ga_slam_visualization/urdf/meshes/exoter/wheel.stl scale=1.66 1 1.66
- link ml_wheel: geometry visual mesh filename=package://ga_slam_visualization/urdf/meshes/exoter/wheel.stl scale=1.66 1 1.66
- link mr_wheel: geometry visual mesh filename=package://ga_slam_visualization/urdf/meshes/exoter/wheel.stl scale=1.66 1 1.66
- link rl_wheel: geometry visual mesh filename=package://ga_slam_visualization/urdf/meshes/exoter/wheel.stl scale=1.66 1 1.66
- link rr_wheel: geometry visual mesh filename=package://ga_slam_visualization/urdf/meshes/exoter/wheel.stl scale=1.66 1 1.66
Joints:
- joint fl_drive: type continuous -> fixed
- joint fl_steer: type continuous -> fixed
- joint fr_drive: type continuous -> fixed
- joint fr_steer: type continuous -> fixed
- joint front_passive: parent body -> body_base; type continuous -> fixed
- joint left_passive: parent body -> body_base; type continuous -> fixed
- joint left_rocker_bogie: type continuous -> fixed
- joint mast_joint: parent body -> body_base
- joint ml_drive: type continuous -> fixed
- joint mr_drive: type continuous -> fixed
- joint pan_joint: type continuous -> fixed
- joint right_passive: parent body -> body_base; type continuous -> fixed
- joint right_rocker_bogie: type continuous -> fixed
- joint rl_drive: type continuous -> fixed
- joint rl_steer: type continuous -> fixed
- joint rr_drive: type continuous -> fixed
- joint rr_steer: type continuous -> fixed
- joint tilt_joint: type continuous -> fixed
